File: carte actionneur.kicad_sch (KiCad schematic)
At the start: 88 parts, among them J1 Conn_01x03_Pin, J10 Conn_01x03_Pin, J11 Conn_01x02, J12 Conn_01x02_Pin, J13 Conn_01x02_Pin, J14 Conn_01x02_Pin, J15 Conn_01x02, J16 Conn_01x02_Pin, J17 Conn_01x04_Pin, J18 Conn_01x02_Pin, J19 Conn_01x04_Pin, J2 Conn_01x02, J20 Conn_01x02_Pin, J21 Conn_01x08_Pin, J22 Conn_01x02_Pin, J23 Conn_01x02_Pin, J24 Conn_01x02_Pin, J25 Conn_01x03_Pin, J26 Conn_01x03_Pin, J27 Conn_01x03_Pin, J28 Conn_01x02_Pin, J3 Conn_01x04_Pin, J4 Conn_01x02_Pin, J4 Connecteur Programmation, J6 Conn_01x08_Pin, J7 Conn_01x03_Pin, J8 Conn_01x03_Pin, J9 Conn_01x03_Pin, Q1 Q_NMOS_GDS, Q2 QM6006D, Q3 QM6006D, Q4 QM6006D, U1 MEGA_PRO_EMBED_CH340G___ATMEG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, U2 YAAJ_DCDC_StepDown_LM2596, U3 ZXBM5210-SP, U4 YAAJ_DCDC_StepDown_LM2596, U5 YAAJ_DCDC_StepDown_LM2596, U7 ZXBM5210-SP

Commit message: dev continues
Parts:
- removed C3, C4: 100nF, Capacitor_SMD:C_0805_2012Metric, symbol Device:C
- removed C7: 100µ, Capacitor_THT:CP_Radial_D8.0mm_P3.50mm, symbol Device:C_Polarized
- removed D3, D4: D, Diode_SMD:D_SOD-123, symbol Device:D
- removed J1, J10, J25, J26, J27, J7, J8, J9: Conn_01x03_Pin, Connector_PinHeader_2.54mm:PinHeader_1x03_P2.54mm_Vertical, symbol Connector:Conn_01x03_Pin
- removed J11: Conn_01x02, Connector_JST:JST_XH_B2B-XH-A_1x02_P2.50mm_Vertical, symbol Connector_Generic:Conn_01x02
- removed J12, J13, J14, J16, J18, J20, J28, J4: Conn_01x02_Pin, Connector_PinHeader_2.54mm:PinHeader_1x02_P2.54mm_Vertical, symbol Connector:Conn_01x02_Pin
- removed J21, J6: Conn_01x08_Pin, Connector_PinHeader_2.54mm:PinHeader_1x08_P2.54mm_Vertical, symbol Connector:Conn_01x08_Pin
- removed J22, J23: Conn_01x02_Pin, Connector_JST:JST_XH_B2B-XH-A_1x02_P2.50mm_Vertical, symbol Connector:Conn_01x02_Pin
- removed JP16, JP17, JP18, JP19, JP20, JP21: Jumper_2_Open, Jumper:SolderJumper-2_P1.3mm_Open_TrianglePad1.0x1.5mm, symbol Jumper:Jumper_2_Open
- removed Q2, Q3: QM6006D, Package_TO_SOT_SMD:TO-252-2, symbol Transistor_FET:QM6006D
- removed R10, R9: 100k, Resistor_SMD:R_0805_2012Metric, symbol Device:R
- removed R4, R5: 10k, Resistor_SMD:R_0805_2012Metric, symbol Device:R
- removed U2, U5: YAAJ_DCDC_StepDown_LM2596, lib-buck-converter:YAAJ_DCDC_StepDown_LM2596, symbol yaaj_dcdc_stepdown_lm2596:YAAJ_DCDC_StepDown_LM2596
- removed U3: ZXBM5210-SP, Package_SO:Diodes_SO-8EP, symbol Driver_Motor:ZXBM5210-SP
- added A4: Pololu_Breakout_A4988, A4988:Pololu_Breakout-16_15.2x20.3mm, symbol Driver_Motor:Pololu_Breakout_A4988
- added C1, C2: 100µ, Capacitor_THT:CP_Radial_D8.0mm_P3.50mm, symbol Device:C_Polarized
- added J1, J4: Conn_01x08_Pin, Connector_PinHeader_2.54mm:PinHeader_1x08_P2.54mm_Vertical, symbol Connector:Conn_01x08_Pin
- added J11: Conn_01x04_Pin, Connector_PinHeader_2.54mm:PinHeader_1x04_P2.54mm_Vertical, symbol Connector:Conn_01x04_Pin
- added J22: Conn_01x04_Pin, Connector_JST:JST_XH_B4B-XH-A_1x04_P2.50mm_Vertical, symbol Connector:Conn_01x04_Pin
- added J6, J7, J8: Conn_01x07_Pin, Connector_PinHeader_2.54mm:PinHeader_1x07_P2.54mm_Vertical, symbol Connector:Conn_01x07_Pin
- added PS1: TEL_15-2411, TEL151211, symbol TEL_15-2411:TEL_15-2411
Connections:
- net Servo8 is gone; now on net ctrlActionneur1: U1.D12
- net +5V: now also JP11.2 (B), JP13.1 (A), JP14.1 (A), JP15.1 (A), JP23.2 (B), A4.2 (VDD), J7.1 (Pin_1), J7.2 (Pin_2), J7.3 (Pin_3), J7.4 (Pin_4), J7.5 (Pin_5), J7.6 (Pin_6), J7.7 (Pin_7), PS1.3 (+VOUT)
- net DIR1: now also A2.16 (DIR); no longer A1.16 (DIR)
- net DIR2: now also A3.16 (DIR); no longer A2.16 (DIR)
- net DIR3: now also A1.16 (DIR); no longer A3.16 (DIR)
- net GND: now also A4.1 (GND), A4.7 (GND), C1.2, C2.2, J11.1 (Pin_1), J4.1 (Pin_1), J4.2 (Pin_2), J4.3 (Pin_3), J4.4 (Pin_4), J4.5 (Pin_5), J4.6 (Pin_6), J4.7 (Pin_7), J4.8 (Pin_8), J8.1 (Pin_1), J8.2 (Pin_2), J8.3 (Pin_3), J8.4 (Pin_4), J8.5 (Pin_5), J8.6 (Pin_6), J8.7 (Pin_7), PS1.2 (-VIN_(GND)), PS1.5 (-VOUT)
- net Reset: now also A4.13 (~{RESET})
- net STEP1: now also A2.15 (STEP); no longer A1.15 (STEP)
- net STEP2: now also A3.15 (STEP); no longer A2.15 (STEP)
- net STEP3: now also A1.15 (STEP); no longer A3.15 (STEP)
- net Servo1: now also J6.1 (Pin_1)
- net Servo2: now also J6.2 (Pin_2)
- net Servo3: now also J6.3 (Pin_3)
- net Servo4: now also J6.4 (Pin_4)
- net Servo5: now also J6.5 (Pin_5)
- net Servo6: now also J6.6 (Pin_6)
- net Servo7: now also J6.7 (Pin_7)
- net Sleep: now also A4.14 (~{SLEEP})
- net VmotDC: no longer JP13.2 (B)
- net ctrlActionneur1: now also Q4.1 (G), R11.1; no longer U1.D4
- net ctrlActionneur3: no longer Q4.1 (G), R11.1
- net Enable4: now reaches U1.D47
- net Enable4: now also A4.9 (~{ENABLE})
- net STEP4: now reaches U1.D49
- net STEP4: now also U1.D4, A4.15 (STEP)
- net DIR4: now reaches U1.D51
- net DIR4: now also A4.16 (DIR)
- net +24V renamed +BATT
- net +BATT: now also A1.8 (VMOT), A2.8 (VMOT), A3.8 (VMOT), C8.1, C9.1, JP12.2 (B), JP24.2 (B), A4.8 (VMOT), C1.1, C2.1, PS1.1 (+VIN_(VCC))
- net +3.3V: no longer names the net of U1.3V3_1 (3V3), U1.3V3_2 (3V3)
- removed net 12V Mot: A1.8 (VMOT), A2.8 (VMOT), A3.8 (VMOT), C8.1, C9.1, JP12.2 (B), JP15.2 (B), JP24.2 (B), U1.VIN_1 (VIN), U1.VIN_2 (VIN)
- removed net 5V Servo: JP11.2 (B), JP14.2 (B), JP23.2 (B)
- net Capt1 renamed Sens1
- net Sens1: now also J1.1 (Pin_1)
- net Capt2 renamed Sens2
- net Sens2: now also J1.2 (Pin_2)
- net Capt3 renamed Sens3
- net Sens3: now also J1.3 (Pin_3)
- net Capt4 renamed Sens4
- net Sens4: now also J1.4 (Pin_4)
- net Capt5 renamed Sens5
- net Sens5: now also J1.5 (Pin_5)
- net Capt6 renamed Sens6
- net Sens6: now also J1.6 (Pin_6)
- net Capt7 renamed Sens7
- net Sens7: now also J1.7 (Pin_7)
- net Capt8 renamed Sens8
- net Sens8: now also J1.8 (Pin_8)
- net FWD2: no longer names the net of U1.D52
- net REV2: no longer names the net of U1.D44
- net ctrlActionneur2: no longer names the net of U1.D42
- new net: U1.VIN_1 (VIN), U1.VIN_2 (VIN)
- new net: A4.10 (MS1), JP13.2 (B)
- new net: A4.11 (MS2), JP14.2 (B)
- new net: A4.12 (MS3), JP15.2 (B)
- new net: A4.3 (1B), J22.4 (Pin_4)
- new net: A4.4 (1A), J22.3 (Pin_3)
- new net: A4.5 (2A), J22.2 (Pin_2)
- new net: A4.6 (2B), J22.1 (Pin_1)
- new net LED_B: J11.4 (Pin_4)
- new net LED_G: J11.3 (Pin_3)
- new net LED_R: J11.2 (Pin_2)
- no-connect marks 23 -> 38
Other:
- note added: "TODO I2C CONN"
- note added: "TODO PWM LIDAR"
- moved on the sheet: A2, A3, C5, C6, C8, C9, D1, D5, H1, H2, H3, J15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

Commit message: presque fini
Parts:
- removed J4: Connecteur Programmation, Connector_PinHeader_2.54mm:PinHeader_1x04_P2.54mm_Vertical, symbol Connector_Generic:Conn_01x04
- removed JP10, JP22: Jumper_2_Open, Jumper:SolderJumper-2_P1.3mm_Open_TrianglePad1.0x1.5mm, symbol Jumper:Jumper_2_Open
- removed U4: YAAJ_DCDC_StepDown_LM2596, lib-buck-converter:YAAJ_DCDC_StepDown_LM2596, symbol yaaj_dcdc_stepdown_lm2596:YAAJ_DCDC_StepDown_LM2596
- added J5: Conn_01x03, Connector_JST:JST_XH_B3B-XH-A_1x03_P2.50mm_Vertical, symbol Connector_Generic:Conn_01x03
- PS1: footprint TEL151211 -> (none)
Connections:
- net ctrlActionneur3 is gone; now on net DIR2: U1.D43
- net +BATT: now also J2.1 (Pin_1); no longer J2.2 (Pin_2)
- net DIR1: now also U1.D42; no longer U1.D25
- net DIR2: no longer U1.D27
- net DIR3: now also U1.D28; no longer U1.D29
- net DIR4: now also U1.D29; no longer U1.D51
- net Enable1: now also U1.D47; no longer U1.D28
- net Enable2: now also U1.D40; no longer U1.D26
- net Enable3: now also U1.D30; no longer U1.D24
- net Enable4: now also U1.D31; no longer U1.D47
- net GND: now also J5.3 (Pin_3)
- net LED_B: now also U1.A10
- net LED_G: now also U1.A11
- net LED_R: now also U1.A12
- net STEP1: now also U1.D2; no longer U1.D3
- net STEP2: now also U1.D3; no longer U1.D2
- net STEP3: now also U1.D4; no longer U1.D5
- net STEP4: now also U1.D5; no longer U1.D4, U1.D49
- net SWCLK: now also J5.1 (Pin_1)
- net SWDIO: now also J5.2 (Pin_2)
- net ctrlActionneur1: now also U1.D44; no longer U1.D12
- net at Q1.2 (D): now also J2.2 (Pin_2); no longer J2.1 (Pin_1)
- no-connect marks 38 -> 34
Other:
- note added: "TODO FUSIBLE"
- note removed: "Borne +"
- note removed: "Borne -"
- note removed: "TODO I2C CONN"
- moved on the sheet: J2, PS1

Commit message: Finished
Parts:
- added F1: Fuse, FuseHolder:FUSE_0154004.DR, symbol Device:Fuse
- added J9: Conn_01x01_Pin, Connector_PinHeader_2.54mm:PinHeader_1x01_P2.54mm_Vertical, symbol Connector:Conn_01x01_Pin
- added TP1: TestPoint, TestPoint:TestPoint_Bridge_Pitch2.0mm_Drill0.7mm, symbol Connector:TestPoint
Connections:
- net +BATT: now also F1.2; no longer J2.1 (Pin_1)
- net FWD1: now also U1.D12; no longer U1.D46
- net GND: now also TP1.1
- new net: F1.1, J2.1 (Pin_1)
- new net PWM_LIDAR: J9.1 (Pin_1), U1.D46
- no-connect marks 34 -> 39
Other:
- note added: "I2C"
- note removed: "TODO FUSIBLE"
- note removed: "TODO PWM LIDAR"
Changed lines of the file:
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@@
   (junction (at 332.105 98.425) (diameter 0) (color 0 0 0 0)
   )
-  (junction (at 79.375 191.77) (diameter 0) (color 0 0 0 0)
-  )
   (junction (at 127 62.23) (diameter 0) (color 0 0 0 0)
   )
+  (junction (at 79.375 191.77) (diameter 0) (color 0 0 0 0)
+  )
   (junction (at 56.515 118.11) (diameter 0) (color 0 0 0 0)
   )
@@
   (no_connect (at 239.395 149.225))
   (no_connect (at 274.955 93.345))
+  (no_connect (at 239.395 106.045))
   (no_connect (at 239.395 57.785))
   (no_connect (at 239.395 159.385))
@@
   (no_connect (at 239.395 93.345))
   (no_connect (at 239.395 133.985))
+  (no_connect (at 274.955 106.045))
   (no_connect (at 239.395 136.525))
   (no_connect (at 239.395 123.825))
@@
   (no_connect (at 274.955 90.805))
   (no_connect (at 239.395 62.865))
+  (no_connect (at 274.955 139.065))
   (no_connect (at 274.955 144.145))
   (no_connect (at 274.955 136.525))
@@
   (no_connect (at 239.395 156.845))
   (no_connect (at 239.395 144.145))
+  (no_connect (at 274.955 103.505))
   (no_connect (at 239.395 151.765))
+  (no_connect (at 239.395 103.505))
   (wire (pts (xy 67.31 209.55) (xy 74.295 209.55))
     (stroke (width 0) (type default))
@@
     (stroke (width 0) (type default))
   )
-  (wire (pts (xy 282.575 88.265) (xy 274.955 88.265))
-    (stroke (width 0) (type default))
-  )
   (wire (pts (xy 283.845 221.615) (xy 291.465 221.615))
     (stroke (width 0) (type default))
   )
-  (wire (pts (xy 231.14 106.045) (xy 239.395 106.045))
-    (stroke (width 0) (type default))
-  )
   (wire (pts (xy 220.98 223.52) (xy 229.235 223.52))
     (stroke (width 0) (type default))
@@
     (stroke (width 0) (type default))
   )
-  (wire (pts (xy 318.135 219.075) (xy 319.405 219.075))
+  (wire (pts (xy 67.31 191.77) (xy 69.85 191.77))
     (stroke (width 0) (type default))
   )
-  (wire (pts (xy 233.68 231.14) (xy 236.855 231.14))
+  (wire (pts (xy 318.135 219.075) (xy 319.405 219.075))
     (stroke (width 0) (type default))
   )
-  (wire (pts (xy 67.31 191.77) (xy 79.375 191.77))
+  (wire (pts (xy 233.68 231.14) (xy 236.855 231.14))
     (stroke (width 0) (type default))
   )
@@
     (stroke (width 0) (type default))
   )
-  (wire (pts (xy 220.98 128.905) (xy 239.395 128.905))
-    (stroke (width 0) (type default))
-  )
   (wire (pts (xy 79.375 199.39) (xy 79.375 201.93))
     (stroke (width 0) (type default))
@@
     (stroke (width 0) (type default))
   )
-  (wire (pts (xy 284.48 103.505) (xy 274.955 103.505))
-    (stroke (width 0) (type default))
-  )
   (wire (pts (xy 86.36 88.9) (xy 86.36 90.17))
     (stroke (width 0) (type default))
@@
     (stroke (width 0) (type default))
   )
-  (wire (pts (xy 284.48 108.585) (xy 274.955 108.585))
-    (stroke (width 0) (type default))
-  )
   (wire (pts (xy 274.955 45.085) (xy 282.575 45.085))
     (stroke (width 0) (type default))
@@
     (stroke (width 0) (type default))
   )
-  (wire (pts (xy 231.14 103.505) (xy 239.395 103.505))
-    (stroke (width 0) (type default))
-  )
   (wire (pts (xy 86.995 209.55) (xy 99.06 209.55))
     (stroke (width 0) (type default))
@@
     (stroke (width 0) (type default))
   )
-  (wire (pts (xy 127 62.23) (xy 127.635 62.23))
+  (wire (pts (xy 77.47 191.77) (xy 79.375 191.77))
     (stroke (width 0) (type default))
   )
-  (wire (pts (xy 281.305 131.445) (xy 274.955 131.445))
+  (wire (pts (xy 127 62.23) (xy 127.635 62.23))
     (stroke (width 0) (type default))
   )
@@
     (stroke (width 0) (type default))
   )
-  (wire (pts (xy 284.48 106.045) (xy 274.955 106.045))
-    (stroke (width 0) (type default))
-  )
   (wire (pts (xy 67.31 59.69) (xy 76.2 59.69))
     (stroke (width 0) (type default))
@@
     (fill (type none))
   )
-  (text "TODO FUSIBLE" (at 69.85 184.15 0)
-    (effects (font (size 1.27 1.27)) (justify left bottom))
-  )
-  (text "TODO PWM LIDAR" (at 302.26 60.96 0)
+  (text "I2C\n" (at 215.9 29.21 0)
     (effects (font (size 1.27 1.27)) (justify left bottom))
   )
@@
     )
   )
-  (global_label "FWD1" (shape input) (at 281.305 131.445 0) (fields_autoplaced)
+  (global_label "PWM_LIDAR" (shape input) (at 274.955 131.445 0) (fields_autoplaced)
     (effects (font (size 1.27 1.27)) (justify left))
-    (property "Intersheetrefs" "${INTERSHEET_REFS}" (at 289.3097 131.445 0)
+    (property "Intersheetrefs" "${INTERSHEET_REFS}" (at 288.3421 131.445 0)
       (effects (font (size 1.27 1.27)) (justify left) hide)
     )
@@
     )
   )
+  (global_label "FWD1" (shape input) (at 274.955 88.265 0) (fields_autoplaced)
+    (effects (font (size 1.27 1.27)) (justify left))
+    (property "Intersheetrefs" "${INTERSHEET_REFS}" (at 282.9597 88.265 0)
+      (effects (font (size 1.27 1.27)) (justify left) hide)
+    )
+  )
   (global_label "DIR2" (shape input) (at 239.395 126.365 180) (fields_autoplaced)
     (effects (font (size 1.27 1.27)) (justify right))
@@
     )
   )
-  (global_label "DIR3" (shape input) (at 284.48 108.585 0) (fields_autoplaced)
+  (global_label "DIR3" (shape input) (at 274.955 108.585 0) (fields_autoplaced)
     (effects (font (size 1.27 1.27)) (justify left))
-    (property "Intersheetrefs" "${INTERSHEET_REFS}" (at 291.8195 108.585 0)
+    (property "Intersheetrefs" "${INTERSHEET_REFS}" (at 282.2945 108.585 0)
       (effects (font (size 1.27 1.27)) (justify left) hide)
     )
@@
     )
   )
+  (global_label "PWM_LIDAR" (shape input) (at 308.61 149.225 0) (fields_autoplaced)
+    (effects (font (size 1.27 1.27)) (justify left))
+    (property "Intersheetrefs" "${INTERSHEET_REFS}" (at 321.9971 149.225 0)
+      (effects (font (size 1.27 1.27)) (justify left) hide)
+    )
+  )
   (global_label "Sens2" (shape input) (at 239.395 113.665 180) (fields_autoplaced)
     (effects (font (size 1.27 1.27)) (justify right))
@@
     )
   )
-  (global_label "REV1" (shape input) (at 220.98 128.905 180) (fields_autoplaced)
+  (global_label "REV1" (shape input) (at 239.395 128.905 180) (fields_autoplaced)
     (effects (font (size 1.27 1.27)) (justify right))
-    (property "Intersheetrefs" "${INTERSHEET_REFS}" (at 213.8498 128.8256 0)
+    (property "Intersheetrefs" "${INTERSHEET_REFS}" (at 232.2648 128.8256 0)
       (effects (font (size 1.27 1.27)) (justify right) hide)
     )
@@
     )
   )
+  (symbol (lib_id "Connector:Conn_01x01_Pin") (at 303.53 149.225 0) (unit 1)
+    (in_bom yes) (on_board yes) (dnp no)
+    (property "Reference" "J9" (at 301.625 149.225 0)
+      (effects (font (size 1.27 1.27)))
+    )
+    (property "Value" "Conn_01x01_Pin" (at 304.165 147.32 0)
+      (effects (font (size 1.27 1.27)) hide)
+    )
+    (property "Footprint" "Connector_PinHeader_2.54mm:PinHeader_1x01_P2.54mm_Vertical" (at 303.53 149.225 0)
+      (effects (font (size 1.27 1.27)) hide)
+    )
+    (property "Datasheet" "~" (at 303.53 149.225 0)
+      (effects (font (size 1.27 1.27)) hide)
+    )
+    (pin "1")
+    (instances
+      (project "carte actionneur"
+        (path "/fdaebf9c-99c5-4ed7-ad84-64cff9929291"
+          (reference "J9") (unit 1)
+        )
+      )
+    )
+  )
   (symbol (lib_id "power:GND") (at 61.595 239.395 0) (unit 1)
     (in_bom yes) (on_board yes) (dnp no) (fields_autoplaced)
@@
     )
   )
+  (symbol (lib_id "Device:Fuse") (at 73.66 191.77 90) (unit 1)
+    (in_bom yes) (on_board yes) (dnp no) (fields_autoplaced)
+    (property "Reference" "F1" (at 73.66 186.69 90)
+      (effects (font (size 1.27 1.27)))
+    )
+    (property "Value" "Fuse" (at 73.66 189.23 90)
+      (effects (font (size 1.27 1.27)))
+    )
+    (property "Footprint" "FuseHolder:FUSE_0154004.DR" (at 73.66 193.548 90)
+      (effects (font (size 1.27 1.27)) hide)
+    )
+    (property "Datasheet" "~" (at 73.66 191.77 0)
+      (effects (font (size 1.27 1.27)) hide)
+    )
+    (pin "1")
+    (pin "2")
+    (instances
+      (project "carte actionneur"
+        (path "/fdaebf9c-99c5-4ed7-ad84-64cff9929291"
+          (reference "F1") (unit 1)
+        )
+      )
+    )
+  )
   (symbol (lib_name "GND_3") (lib_id "power:GND") (at 323.85 137.795 0) (unit 1)
     (in_bom yes) (on_board yes) (dnp no) (fields_autoplaced)
@@
     )
   )
+  (symbol (lib_id "power:GND") (at 104.14 238.125 180) (unit 1)
+    (in_bom yes) (on_board yes) (dnp no) (fields_autoplaced)
+    (property "Reference" "#PWR09" (at 104.14 231.775 0)
+      (effects (font (size 1.27 1.27)) hide)
+    )
+    (property "Value" "GND" (at 104.14 233.68 0)
+      (effects (font (size 1.27 1.27)))
+    )
+    (property "Footprint" "" (at 104.14 238.125 0)
+      (effects (font (size 1.27 1.27)) hide)
+    )
+    (property "Datasheet" "" (at 104.14 238.125 0)
+      (effects (font (size 1.27 1.27)) hide)
+    )
+    (pin "1")
+    (instances
+      (project "carte actionneur"
+        (path "/fdaebf9c-99c5-4ed7-ad84-64cff9929291"
+          (reference "#PWR09") (unit 1)
+        )
+      )
+    )
+  )
   (symbol (lib_id "Device:C") (at 299.085 202.565 0) (unit 1)
     (in_bom yes) (on_board yes) (dnp no) (fields_autoplaced)
@@
         )
       )
+    )
+  )
+  (symbol (lib_id "Connector:TestPoint") (at 104.14 238.125 180) (unit 1)
+    (in_bom yes) (on_board yes) (dnp no) (fields_autoplaced)
+    (property "Reference" "TP1" (at 106.68 240.157 0)
+      (effects (font (size 1.27 1.27)) (justify right))
+    )
+    (property "Value" "TestPoint" (at 106.68 242.697 0)
+      (effects (font (size 1.27 1.27)) (justify right))
+    )
+    (property "Footprint" "TestPoint:TestPoint_Bridge_Pitch2.0mm_Drill0.7mm" (at 99.06 238.125 0)
+      (effects (font (size 1.27 1.27)) hide)
+    )
+    (property "Datasheet" "~" (at 99.06 238.125 0)
+      (effects (font (size 1.27 1.27)) hide)
+    )
+    (pin "1")
+    (instances
+      (project "carte actionneur"
+        (path "/fdaebf9c-99c5-4ed7-ad84-64cff9929291"
+          (reference "TP1") (unit 1)
+        )
+      )
