File: carte actionneur.kicad_sch (KiCad schematic)
At the start: 58 parts, among them J1 Conn_01x08_Pin, J10 Conn_01x08_Pin, J11 Conn_01x04_Pin, J15 Conn_01x02, J17 Conn_01x04_Pin, J19 Conn_01x04_Pin, J2 Conn_01x02, J22 Conn_01x04_Pin, J3 Conn_01x04_Pin, J4 Conn_01x08_Pin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

Commit message: second
Parts:
- removed C10: 680uF, symbol Device:C_Polarized_US
- removed C11: 220uF, symbol Device:C_Polarized_US
- removed D2: 1N5824, Diode_THT:D_DO-201AD_P15.24mm_Horizontal, symbol Diode:1N5822
- removed R1: 10k, Resistor_SMD:R_0805_2012Metric, symbol Device:R
- removed U3: LM2596S-5, Package_TO_SOT_SMD:TO-263-5_TabPin3, symbol Regulator_Switching:LM2596S-5
- added C10, C11, C14: 22u, Capacitor_SMD:C_1206_3216Metric, symbol Device:C_Polarized_Small
- added C12: 1u, Capacitor_SMD:C_1206_3216Metric, symbol Device:C_Polarized_Small
- added C13: 1u, Capacitor_SMD:C_1206_3216Metric, symbol Device:C_Small
- added C7: 100n, Capacitor_SMD:C_1206_3216Metric, symbol Device:C_Small
- added JP10: Jumper_2_Open, Jumper:SolderJumper-2_P1.3mm_Open_TrianglePad1.0x1.5mm, symbol Jumper:Jumper_2_Open
- added R1: 10, Resistor_SMD:R_1206_3216Metric, symbol Device:R_Small
- added R2: 100k, Resistor_SMD:R_1206_3216Metric, symbol Device:R_Small
- added R3: 13.7k, Resistor_SMD:R_1206_3216Metric, symbol Device:R_Small
- added U3: MP2236CGJ-P, Package_TO_SOT_SMD:TSOT-23-8, symbol MP2236:MP2236CGJ-P
- C4: value 100u -> 22uF; footprint (none) -> Capacitor_SMD:C_1206_3216Metric
- L2: value 33uH -> 3.3uH; footprint (none) -> Inductor_SMD:L_Coilcraft_XAL6030-XXX
Connections:
- net +5V: now also C11.1, C14.1, R2.1
- net +5VD: now also JP10.2 (B)
- net +BATT: now also C10.1, C12.1, U3.2 (IN)
- net GND: now also C10.2, C11.2, C12.2, C13.2, C14.2, R3.2, U3.1 (AGND), U3.4 (GND)
- net POW_EN: now also JP10.1 (A), U3.6 (EN)
- net at L2.1: now also C7.2, U3.3 (SW)
- new net: R1.1, U3.5 (BST)
- new net: C7.1, R1.2
- new net: R2.2, R3.1, U3.8 (FB)
- new net: C13.1, U3.7 (VCC)
Other:
- note added: "18Vin 6A 5V Sync Buck Converter"
- note added: "1A 5V Buck Converter"
- moved on the sheet: L2
