File: carte actionneur.kicad_sch (KiCad schematic)
At the start: 64 parts, among them J1 Conn_01x08_Pin, J10 Conn_01x08_Pin, J11 Conn_01x04_Pin, J15 Conn_01x02, J17 Conn_01x04_Pin, J19 Conn_01x04_Pin, J2 Conn_01x02, J22 Conn_01x04_Pin, J3 Conn_01x04_Pin, J4 Conn_01x08_Pin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

Commit message: final rev2
Parts:
- removed JP23, JP24: Jumper_2_Open, Jumper:SolderJumper-2_P1.3mm_Open_TrianglePad1.0x1.5mm, symbol Jumper:Jumper_2_Open
- removed R6, R7: 10k, Resistor_SMD:R_0805_2012Metric, symbol Device:R
- removed U7: ZXBM5210-SP, Package_SO:Diodes_SO-8EP, symbol Driver_Motor:ZXBM5210-SP
- added U4: DRV8870DDA, Package_SO:Texas_HTSOP-8-1EP_3.9x4.9mm_P1.27mm_EP2.95x4.9mm_Mask2.4x3.1mm_ThermalVias, symbol Driver_Motor:DRV8870DDA
- R3: footprint Resistor_SMD:R_1206_3216Metric -> Resistor_SMD:R_0805_2012Metric
Connections:
- net +5VD: now also U4.4 (VREF)
- net +BATT: now also C3.1, C6.1, U4.5 (VM)
- net FWD1: now also U1.D44, U4.3 (IN1); no longer U1.D12
- net GND: now also U4.1 (GND), U4.7 (ISEN), U4.9 (GND)
- net POW_EN: now also U1.D14
- net REV1: now also U4.2 (IN2)
- net at J15.1 (Pin_1): now also U4.6 (OUT1)
- net at J15.2 (Pin_2): now also U4.8 (OUT2)
Other:
- note added: "DC MOTOR DRIVER H-BRIDGE 3.6A"
- moved on the sheet: C3, C6, F1, J1, J10, J15, J2, J4, J9
