File: carte actionneur.kicad_pcb (KiCad board)
At the start: 2 copper layers, 87.5 x 90 mm, 103 parts, among them J1 Conn_01x08_Pin, J11 Conn_01x04_Pin, J15 Conn_01x02, J17 Conn_01x04_Pin, J19 Conn_01x04_Pin, J2 Conn_01x02, J22 Conn_01x04_Pin, J24 Conn_01x02_Pin, J3 Conn_01x04_Pin, J4 Conn_01x08_Pin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

Commit message: first
Parts:
- removed D1: D_Zener, Diode_SMD:D_SOD-123
- removed D5: D, Diode_SMD:D_SOD-123
- removed J24: Conn_01x02_Pin, Connector_JST:JST_XH_B2B-XH-A_1x02_P2.50mm_Vertical
- removed JP11, JP12: Jumper_2_Open, Jumper:SolderJumper-2_P1.3mm_Open_TrianglePad1.0x1.5mm
- removed PS1: TEL_15-2411, TEL_15-2411:TEL151211
- removed Q1: Q_NMOS_GDS, Package_TO_SOT_SMD:TO-252-2
- removed Q4: QM6006D, Package_TO_SOT_SMD:TO-252-2
- removed R11: 100k, Resistor_SMD:R_0805_2012Metric
- removed REF** (x2): LOGO, Silkscreen:LOGO
- removed REF**: Microsteps, Silkscreen:Microsteps
- removed the kibuzzard-679FD879 at (115.5, 116.8)
- removed the kibuzzard-679FD896 at (118.5, 116.3)
- removed kibuzzard-67A145CB: G***, kibuzzard-67A145CB
- added C3: 100µ, Capacitor_THT:CP_Radial_D8.0mm_P3.50mm, F.Cu at (74.5, 117.6)
- added D2: 1N5824, Diode_THT:D_DO-201AD_P15.24mm_Horizontal, F.Cu at (34.4, 119.6)
- added J10: Conn_01x08_Pin, Connector_PinHeader_2.54mm:PinHeader_1x08_P2.54mm_Vertical, F.Cu at (109.8, 88.1)
- added U2: 173010542, MagIC_THT_Wurth:U_Wurth_MagIC-FDSM_173010x42, F.Cu at (166.1, 134.5)
- added U3: LM2596S-5, Package_TO_SOT_SMD:TO-263-5_TabPin3, F.Cu at (64.6, 111.5)
- R1: value 56k -> 10k; footprint Resistor_SMD:R_0805_2012Metric_Pad1.20x1.40mm_HandSolder -> Resistor_SMD:R_0805_2012Metric; moved to F.Cu
- moved R1 87.3 mm to (50.8, 107.9)
Connections:
- A1 pad 2: +5V -> +5VD
- A2 pad 2: +5V -> +5VD
- A3 pad 2: +5V -> +5VD
- A4 pad 2: +5V -> +5VD
- C5 pad 1: +5V -> +5VD
- J2 pad 2: Net-(J2-Pin_2) -> GND
- JP1 pad 1: +5V -> +5VD
- JP13 pad 1: +5V -> +5VD
- JP14 pad 1: +5V -> +5VD
- JP15 pad 1: +5V -> +5VD
- JP2 pad 1: +5V -> +5VD
- JP3 pad 1: +5V -> +5VD
- JP4 pad 1: +5V -> +5VD
- JP5 pad 1: +5V -> +5VD
- JP6 pad 1: +5V -> +5VD
- JP7 pad 1: +5V -> +5VD
- JP8 pad 1: +5V -> +5VD
- JP9 pad 1: +5V -> +5VD
- R1 pad 1: +BATT -> POW_EN
- R1 pad 2: Net-(D1-K) -> GND
- U1 pad 5V_1: +5V -> +5VD
- U1 pad 5V_2: +5V -> +5VD
- U1 pad D44: ctrlActionneur1 -> unconnected-(U1-PadD44)
- U7 pad 3: +5V -> +5VD
- U7 pad 6: +5V -> +5VD
Routing:
- net +5V: track 306.2 -> 239.0 mm
- net ctrlActionneur1: track 31.0 -> 0.00 mm
- net Net-(D1-K): track 15.8 -> 0.00 mm
- net Net-(D5-K): track 14.7 -> 0.00 mm
- net +BATT: track 302.4 -> 288.8 mm
- net Net-(J2-Pin_2): track 10.6 -> 0.00 mm
- net +5VD: track 0.00 -> 7.96 mm
- net Net-(D5-A): track 6.65 -> 0.00 mm
- net REV1: track 64.9 -> 71.1 mm
- net GND: track 187.9 -> 185.0 mm, vias 180 -> 121
Other:
- board text added: "Carte Actionneurs Arduino Ludovic Bouchard Rev2 04/2025"
- board text removed: "+"
- board text removed: "-"
- board text removed: "Carte Actionneurs Arduino Ludovic Bouchard Rev1 02/2025"

Commit message: second
Parts:
- removed D2: 1N5824, Diode_THT:D_DO-201AD_P15.24mm_Horizontal
- added C10: 22u, Capacitor_SMD:C_1206_3216Metric, F.Cu at (150.5, 120.9)
- added C11: 22u, Capacitor_SMD:C_1206_3216Metric, F.Cu at (157.0, 119.4)
- added C12: 1u, Capacitor_SMD:C_1206_3216Metric, F.Cu at (150.5, 118.4)
- added C13: 1u, Capacitor_SMD:C_1206_3216Metric, F.Cu at (150.5, 114.4)
- added C14: 22u, Capacitor_SMD:C_1206_3216Metric, F.Cu at (154.5, 119.4)
- added C4: 22uF, Capacitor_SMD:C_1206_3216Metric, B.Cu at (163.5, 133.0)
- added C7: 100n, Capacitor_SMD:C_1206_3216Metric, F.Cu at (160.5, 112.3)
- added JP10: Jumper_2_Open, Jumper:SolderJumper-2_P1.3mm_Open_TrianglePad1.0x1.5mm, B.Cu at (167.5, 114.0)
- added L2: 3.3uH, Inductor_SMD:L_Coilcraft_XAL6030-XXX, F.Cu at (162.0, 118.4)
- added R2: 100k, Resistor_SMD:R_1206_3216Metric, F.Cu at (152.5, 106.9)
- added R3: 13.7k, Resistor_SMD:R_1206_3216Metric, F.Cu at (151.1, 110.9)
- R1: value 10k -> 10; footprint Resistor_SMD:R_0805_2012Metric -> Resistor_SMD:R_1206_3216Metric
- U3: value LM2596S-5 -> MP2236CGJ-P; footprint Package_TO_SOT_SMD:TO-263-5_TabPin3 -> Package_TO_SOT_SMD:TSOT-23-8
- moved R1 106.2 mm to (157.0, 110.9)
- moved U3 89.5 mm to (154.0, 114.4), turned to 90 degrees
- moved J10 17.1 mm to (126.9, 88.0)
- moved J9 12.8 mm to (121.9, 83.8)
- moved kibuzzard-67A14A78 12.8 mm to (117.1, 83.8)
- moved C3 11.0 mm to (68.8, 127.0)
- moved kibuzzard-679EA236 2.50 mm to (129.5, 109.5)
- moved kibuzzard-679FD606 2.45 mm to (124.5, 105.8)
- moved kibuzzard-679FD637 2.45 mm to (124.5, 103.2)
- moved kibuzzard-679FD63B 2.45 mm to (124.5, 100.7)
- moved kibuzzard-679FD63E 2.45 mm to (124.5, 98.2)
- moved kibuzzard-679FD642 2.45 mm to (124.5, 95.6)
- moved kibuzzard-679FD645 2.45 mm to (124.5, 93.1)
- moved kibuzzard-679FD648 2.45 mm to (124.5, 90.5)
- moved kibuzzard-679FD64B 2.45 mm to (124.5, 88.0)
Connections:
- R1 pad 1: POW_EN -> Net-(U3-BST)
- R1 pad 2: GND -> Net-(C7-Pad1)
- U1 pad RX: unconnected-(U1-PadRX) -> (no net)
- U1 pad TX: unconnected-(U1-PadTX) -> (no net)
- U3 pad 1: +BATT -> GND
- U3 pad 2: Net-(D2-K) -> +BATT
- U3 pad 3: GND -> Net-(U3-SW)
- U3 pad 4: +5V -> GND
- U3 pad 5: POW_EN -> Net-(U3-BST)
Routing:
- net +5VD: track 7.96 -> 274.8 mm, vias 0 -> 7
- net +5V: track 239.0 -> 86.2 mm, vias 9 -> 3
- net POW_EN: track 0.00 -> 27.1 mm, vias 0 -> 1
- net GND: track 185.0 -> 210.7 mm, vias 121 -> 141
- net +BATT: track 288.8 -> 309.1 mm, vias 12 -> 13
- net Net-(U3-SW): track 0.00 -> 12.2 mm
- net PWM_LIDAR: track 26.9 -> 19.1 mm
- net Net-(U3-FB): track 0.00 -> 5.08 mm
- net Net-(U3-VCC): track 0.00 -> 4.66 mm
- net Net-(U3-BST): track 0.00 -> 2.58 mm
- net Net-(C7-Pad1): track 0.00 -> 2.08 mm
- net REV1: track 71.1 -> 72.1 mm
- added copper zone on F.Cu, net Net-(U3-SW)
